File: Plane/Plane.kicad_pcb (KiCad board)
At the start: 2 copper layers, 0 parts

Commit message: init board
Parts:
- added A1: RaspberryPi_Pico, Module:RaspberryPi_Pico_Common_Unspecified, F.Cu at (209.6, 105.3)
- added C1: C_Polarized, Capacitor_THT:CP_Radial_D6.3mm_P2.50mm, F.Cu at (195.6, 48.8)
- added D1: LED, Connector_JST:JST_PH_B2B-PH-K_1x02_P2.00mm_Vertical, F.Cu at (192.0, 105.5)
- added D2: LED, Connector_JST:JST_PH_B2B-PH-K_1x02_P2.00mm_Vertical, F.Cu at (225.5, 106.0)
- added J1: SPI Bus 17, Connector_JST:JST_PH_B6B-PH-K_1x06_P2.00mm_Vertical, F.Cu at (124.5, 112.2)
- added J2: SPI Bus 5, Connector_JST:JST_PH_B6B-PH-K_1x06_P2.00mm_Vertical, F.Cu at (144.4, 108.7)
- added M1: Aileron_Left, Connector_JST:JST_PH_B3B-PH-K_1x03_P2.00mm_Vertical, F.Cu at (226.1, 117.3)
- added M2: Aileron_Right, Connector_JST:JST_PH_B3B-PH-K_1x03_P2.00mm_Vertical, F.Cu at (193.6, 113.3)
- added M3: Elevator, Connector_JST:JST_PH_B3B-PH-K_1x03_P2.00mm_Vertical, F.Cu at (222.6, 74.3)
- added M4: Rudder, Connector_JST:JST_PH_B3B-PH-K_1x03_P2.00mm_Vertical, F.Cu at (192.6, 72.3)
- added M5: Speed Controller, Connector_JST:JST_PH_B3B-PH-K_1x03_P2.00mm_Vertical, F.Cu at (220.2, 138.5)
- added M6: Unassigned, Connector_JST:JST_PH_B3B-PH-K_1x03_P2.00mm_Vertical, F.Cu at (134.5, 101.5)
- added M7: Unassigned, Connector_JST:JST_PH_B3B-PH-K_1x03_P2.00mm_Vertical, F.Cu at (134.6, 91.0)
- added R1: R, Resistor_THT:R_Axial_DIN0309_L9.0mm_D3.2mm_P12.70mm_Horizontal, F.Cu at (155.8, 43.3)
- added R2: R, Resistor_THT:R_Axial_DIN0309_L9.0mm_D3.2mm_P12.70mm_Horizontal, F.Cu at (154.9, 59.3)
- added R3: 10k, Resistor_THT:R_Axial_DIN0309_L9.0mm_D3.2mm_P12.70mm_Horizontal, F.Cu at (170.3, 43.5)
- added R4: R, Resistor_THT:R_Axial_DIN0309_L9.0mm_D3.2mm_P12.70mm_Horizontal, F.Cu at (163.5, 102.3)
- added R5: R, Resistor_THT:R_Axial_DIN0309_L9.0mm_D3.2mm_P12.70mm_Horizontal, F.Cu at (248.1, 92.7)
- added U1: Left Ranging, Connector_JST:JST_PH_B4B-PH-K_1x04_P2.00mm_Vertical, F.Cu at (226.1, 129.3)
- added U10: I2C, Connector_JST:JST_PH_B4B-PH-K_1x04_P2.00mm_Vertical, F.Cu at (234.9, 47.7)
- added U11: PitotPX4, Connector_JST:JST_PH_B4B-PH-K_1x04_P2.00mm_Vertical, F.Cu at (205.7, 144.0)
- added U2: Right Ranging, Connector_JST:JST_PH_B4B-PH-K_1x04_P2.00mm_Vertical, F.Cu at (193.6, 123.3)
- added U3: PX4TelemRadio, Connector_JST:JST_GH_SM06B-GHS-TB_1x06-1MP_P1.25mm_Horizontal, F.Cu at (204.6, 48.8)
- added U4: TBD Ranging, Connector_JST:JST_PH_B4B-PH-K_1x04_P2.00mm_Vertical, F.Cu at (231.1, 137.7)
- added U5: IMU, Connector_JST:JST_PH_B4B-PH-K_1x04_P2.00mm_Vertical, F.Cu at (235.1, 56.3)
- added U6: Baro, Connector_JST:JST_PH_B4B-PH-K_1x04_P2.00mm_Vertical, F.Cu at (235.1, 62.8)
- added U7: MissionComputerSerial, Connector_JST:JST_GH_SM06B-GHS-TB_1x06-1MP_P1.25mm_Horizontal, F.Cu at (190.6, 142.3)
- added U8: TPS2117DRLR, Package_TO_SOT_SMD:SOT-583-8, F.Cu at (162.3, 49.4)
Other:
- board outline added: 85 x 85.5 mm

Commit message: swap resistors to 0805, move stuff around
Parts:
- R1, R2, R3, R4, R5: footprint Resistor_THT:R_Axial_DIN0309_L9.0mm_D3.2mm_P12.70mm_Horizontal -> Resistor_SMD:R_0805_2012Metric_Pad1.20x1.40mm_HandSolder
- moved U10 102.2 mm to (186.0, 137.5), turned to 180 degrees
- moved U5 84.3 mm to (225.0, 140.0), turned to 180 degrees
- moved J2 83.0 mm to (218.1, 147.0)
- moved J1 73.0 mm to (188.6, 147.0)
- moved M7 58.7 mm to (185.0, 121.0), turned to 180 degrees
- moved M5 51.4 mm to (185.0, 101.0), turned to 180 degrees
- moved M6 51.2 mm to (185.0, 110.0), turned to 180 degrees
- moved R1 47.9 mm to (177.5, 86.0)
- moved U8 46.1 mm to (180.0, 92.0)
- moved R3 44.1 mm to (182.0, 86.0)
- moved C1 44.0 mm to (190.0, 92.5), turned to 0 degrees
- moved R2 43.4 mm to (184.0, 91.5)
- moved U6 39.9 mm to (231.0, 102.5), turned to 180 degrees
- moved M4 39.2 mm to (229.0, 87.0), turned to 180 degrees
- moved U3 38.8 mm to (190.5, 85.0), turned to 180 degrees
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Other:
- board size 85 x 85.5 mm -> 58 x 71.5 mm

Commit message: design 1
Parts:
- M5: value Speed Controller -> ESC
- moved J2 10.4 mm to (228.5, 148.0), turned to 180 degrees
- moved R5 7.89 mm to (225.2, 113.0), turned to -90 degrees
- moved U1 5.22 mm to (225.0, 127.0), turned to 0 degrees
- moved D2 4.66 mm to (231.0, 110.0), turned to 180 degrees
- moved M3 4.03 mm to (227.0, 92.0), turned to 0 degrees
- moved M4 4.03 mm to (227.0, 83.5), turned to 0 degrees
- moved U10 2.55 mm to (186.5, 140.0)
- moved R1 2.33 mm to (179.5, 87.2)
- moved M1 2.06 mm to (227.0, 118.0), turned to 0 degrees
- moved R2 1.35 mm to (183.1, 90.5)
- moved U8 1.35 mm to (179.1, 91.0), turned to 180 degrees
- moved R3 1.10 mm to (182.0, 87.1), turned to 90 degrees
- moved U6 1.00 mm to (231.0, 101.5)
Connections:
- A1 pad 2: /radio_rx_mcu_rx -> /radio_tx_mcu_rx
Routing:
- net /VUSB: track 0.00 -> 131.0 mm
- net /i2c_sda: track 0.00 -> 121.4 mm
- net /i2c_scl: track 0.00 -> 106.8 mm, vias 0 -> 1
- net /spi_cs_5: track 0.00 -> 63.1 mm, vias 0 -> 2
- net /spi_clock: track 0.00 -> 62.9 mm
- net /spi_mosi: track 0.00 -> 62.0 mm
- net +5V: track 0.00 -> 59.3 mm, vias 0 -> 7
- net GND: track 0.00 -> 59.2 mm, vias 0 -> 5
- net /range_1_trig: track 0.00 -> 55.7 mm
- net /range_3_trig: track 0.00 -> 54.5 mm
- net /spi_miso: track 0.00 -> 51.9 mm
- net /range_2_echo: track 0.00 -> 41.5 mm
- net /aileron_left: track 0.00 -> 40.8 mm
- net /mission_tx_mcu_rx: track 0.00 -> 36.9 mm
- net /rudder: track 0.00 -> 35.9 mm
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- added copper zone on F.Cu, net +5V
- added copper zone on B.Cu, net GND
Other:
- outline, holes or cut-outs redrawn
