File: Plane/_autosave-Plane.kicad_sch (KiCad schematic)
At the start: 28 parts, among them J1 SPI Bus 17, J2 SPI Bus 5, M1 Aileron_Left, M2 Aileron_Right, M3 Elevator, M4 Rudder, M5 Speed Controller, M6 Unassigned, M7 Unassigned, U1 Left Ranging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

Commit message: design 1
Parts:
- M5: value Speed Controller -> ESC
Changed lines of the file:
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@@
 			)
 		)
-		(property "Value" "Speed Controller"
+		(property "Value" "ESC"
 			(at 125.73 121.4868 0)
 			(effects
